Commit message: created panda_arm_custom.urdf with collision spheres & updated the EE as the net

File: ball.urdf (robot description, URDF)
Before this commit: robot Ball, 1 links, 0 joints
Links:
- link base: geometry visual sphere radius=.03

File: panda_arm_custom.urdf (robot description, URDF)
Before this commit: robot panda, 10 links, 9 joints
Links:
- link panda_link0: geometry collision sphere radius=0.14; visual mesh filename=package://drake_models/franka_description/meshes/visual/lin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
- link panda_link1: geometry collision sphere radius=0.150; visual mesh filename=package://drake_models/franka_description/meshes/visual/lin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
- link panda_link2: geometry collision sphere radius=0.150; visual mesh filename=package://drake_models/franka_description/meshes/visual/lin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
- link panda_link3: geometry collision sphere radius=0.140; visual mesh filename=package://drake_models/franka_description/meshes/visual/lin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
- link panda_link4: geometry collision sphere radius=0.140; visual mesh filename=package://drake_models/franka_description/meshes/visual/lin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
- link panda_link5: geometry collision sphere radius=0.1; collision sphere radius=0.115
- link panda_link6: geometry collision sphere radius=0.11; visual mesh filename=package://drake_models/franka_description/meshes/visual/lin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
- link panda_link7: geometry collision sphere radius=0.08; visual mesh filename=package://drake_models/franka_description/meshes/visual/lin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
- link panda_link8: geometry collision sphere radius=0.03
- link panda_link9: mass None -> 0.07; geometry collision sphere radius=0.085; visual mesh filename=./net3d_2.obj
Joints:
- joint panda_joint9: origin xyz=0 0 0 rpy=0 0 0 -> xyz=0.145 0.145 0.02 rpy=0 0 0

Commit message: added multiple obstacle avoidance

File: ball.urdf (robot description, URDF)
Before this commit: robot Ball, 1 links, 0 joints
Links:
- link base: mass 1 -> 0

File: obstacle.urdf (robot description, URDF)
Before this commit: robot Ball, 1 links, 0 joints
Links:
- removed link base_obs
- added link obs_0, mass 0; visual sphere radius=0.08
- added link obs_1, mass 0; visual sphere radius=0.08
